Commit message: stable_version

File: src/fishbot_description/urdf/first_robot.urdf (robot description, URDF)
Before this commit: robot first_robot, 2 links, 1 joints
Joints:
- joint imu_joint: origin xyz=0.0 0.0 0.003 rpy=0.0 0.0 0.0 -> xyz=0 0 0.03 rpy=0 0 0

File: src/fishbot_description/urdf/fishbot/base.urdf.xacro (robot description, xacro)
@@ -1,35 +1,33 @@
 <?xml version="1.0"?>
-<robot xmlns:xacro="http://www.ros.org/wiki/xacro" >
-    <xacro:include filename="$(find fishbot_description)/urdf/fishbot/common_inertia.xacro" />
-    <xacro:macro name="base_xacro" params="radius length ">
-        <link name="base_footprint"/>
+<robot xmlns:xacro="http://www.ros.org/wiki/xacro">
+   <xacro:include filename="$(find fishbot_description)/urdf/fishbot/common_inertia.xacro" />
+    <xacro:macro name="base_xacro" params="length radius">
+     <link name="base_footprint" />
+        <joint name="base_joint" type="fixed">
+            <parent link="base_footprint" />
+            <child link="base_link" />
+            <origin xyz="0.0 0.0 ${length/2.0+0.032-0.001}" rpy="0 0 0" />
+        </joint>
         <link name="base_link">
-        <collision>
-                        <!-- 沿自己几何中心的偏移与旋转量 -->
-            <origin xyz="0.0 0.0 0.0" rpy="0.0 0.0 0.0"/>
-            <geometry>
-                <cylinder radius="${radius}" length="${length}"/>
-            </geometry>
-            <material name="white">
-                <color rgba="1.0 1.0 1.0 0.5"/>
-            </material>
-        </collision>
-        <visual>
-            <!-- 沿自己几何中心的偏移与旋转量 -->
-            <origin xyz="0.0 0.0 0.0" rpy="0.0 0.0 0.0"/>
-            <geometry>
-                <cylinder radius="${radius}" length="${length}"/>
-            </geometry>
-            <material name="white">
-                <color rgba="1.0 1.0 1.0 0.5"/>
-            </material>
-        </visual>
-        <xacro:cylinder_inertia m="1.0" r="${radius}" h="${length}" />
+            <visual>
+                <origin xyz="0 0 0.0" rpy="0 0 0" />
+                <geometry>
+                    <cylinder length="${length}" radius="${length}" />
+                </geometry>
+                <material name="blue">
+                    <color rgba="0.1 0.1 1.0 0.5"/>
+                </material>
+            </visual>
+            <collision>
+                <origin xyz="0 0 0.0" rpy="0 0 0" />
+                <geometry>
+                    <cylinder length="${length}" radius="${length}" />
+                </geometry>
+                <material name="blue">
+                    <color rgba="0.1 0.1 1.0 0.5"/>
+                </material>
+            </collision>
+            <xacro:cylinder_inertia m="1.0" r="${radius}" h="${length}"/>
         </link>
-    <joint name="joint_name" type="fixed">
-        <origin xyz="0.0 0.0 ${length/2.0+0.032-0.001}"  rpy="0.0 0.0 0.0"/>
-        <parent link="base_footprint"/>
-        <child link="base_link"/>
-    </joint>
     </xacro:macro>
 </robot>

File: src/fishbot_description/urdf/fishbot/fishbot.ros2_control.xacro (robot description, xacro)
@@ -33,11 +33,11 @@
             </joint>
         </ros2_control>
-<gazebo>
+        <gazebo>
         <plugin filename="libgazebo_ros2_control.so" name="gazebo_ros2_control">
             <parameters>$(find fishbot_description)/config/fishbot_ros2_controller.yaml</parameters>
-                <ros>
-                    <remapping>/fishbot_diff_drive_controller/cmd_vel_unstamped:=/cmd_vel</remapping>
-                    <remapping>/fishbot_diff_drive_controller/odom:=/odom</remapping>
-                </ros>
+            <ros>
+                <remapping>/fishbot_diff_drive_controller/cmd_vel_unstamped:=/cmd_vel</remapping>
+                <remapping>/fishbot_diff_drive_controller/odom:=/odom</remapping>
+            </ros>
         </plugin>
 </gazebo>

File: src/fishbot_description/urdf/fishbot/fishbot.urdf.xacro (robot description, xacro)
@@ -1,27 +1,28 @@
 <?xml version="1.0"?>
 <robot xmlns:xacro="http://www.ros.org/wiki/xacro" name="fishbot">
-<!-- 机器人底盘 -->
-<xacro:include filename="$(find fishbot_description)/urdf/fishbot/base.urdf.xacro" />
-<!-- 机器人传感器 -->
-<xacro:include filename="$(find fishbot_description)/urdf/fishbot/sensor/camera.urdf.xacro" />
-<xacro:include filename="$(find fishbot_description)/urdf/fishbot/sensor/laser.urdf.xacro" />
-<xacro:include filename="$(find fishbot_description)/urdf/fishbot/sensor/imu.urdf.xacro" />
-<!-- 机器人轮子 -->
-<xacro:include filename="$(find fishbot_description)/urdf/fishbot/sensor/actuator/wheel.urdf.xacro" />
-<xacro:include filename="$(find fishbot_description)/urdf/fishbot/sensor/actuator/caster.urdf.xarcro" />
-<!-- 机器人控制插件 -->
-<!-- <xacro:include filename="$(find fishbot_description)/urdf/fishbot/plugins/gazebo_control_plugin.xacro" /> -->
-<xacro:include filename="$(find fishbot_description)/urdf/fishbot/plugins/gazebo_sensor_plugin.xacro" />
-<xacro:include filename="$(find fishbot_description)/urdf/fishbot/fishbot.ros2_control.xacro" />
-<xacro:base_xacro radius="0.1" length="0.12" />
-<xacro:imu_xacro xyz="0.0 0.0 0.02"/>
-<xacro:camera_xacro xyz="0.10 0.0 0.075"/>
-<xacro:laser_xacro xyz="-0.00 0.0 0.11"/>
-<xacro:wheel_xacro wheel_name="left_wheel" xyz="0.0 0.1 -0.06"/>
-<xacro:wheel_xacro wheel_name="right_wheel" xyz="0.0 -0.1 -0.06"/>
-<xacro:caster_xacro caster_name="front_caster" xyz="0.08 0.0 -0.076"/>
-<xacro:caster_xacro caster_name="rear_caster" xyz="-0.08 0.0 -0.076"/>
-<!-- <xacro:gazebo_control_plugin /> -->
-<xacro:gazebo_sensor_plugin />
-<xacro:fishbot_ros2_control />
+    <xacro:include filename="$(find fishbot_description)/urdf/fishbot/base.urdf.xacro" />
+    <!-- 传感器组件 -->
+    <xacro:include filename="$(find fishbot_description)/urdf/fishbot/sensor/imu.urdf.xacro" />
+    <xacro:include filename="$(find fishbot_description)/urdf/fishbot/sensor/laser.urdf.xacro" />
+    <xacro:include filename="$(find fishbot_description)/urdf/fishbot/sensor/camera.urdf.xacro" />
+     <!-- 执行器组件 -->
+    <xacro:include filename="$(find fishbot_description)/urdf/fishbot/actuator/wheel.urdf.xacro" />
+    <xacro:include filename="$(find fishbot_description)/urdf/fishbot/actuator/caster.urdf.xacro" />
+    <xacro:base_xacro length="0.12" radius="0.1" />
+    <!-- 传感器 -->
+    <xacro:imu_xacro xyz="0 0 0.02" />
+    <xacro:laser_xacro xyz="0 0 0.10" />
+    <xacro:camera_xacro xyz="0.10 0 0.075" />
+    <!-- 执行器主动轮+从动轮 -->
+    <xacro:wheel_xacro wheel_name="left" xyz="0 0.10 -0.06" />
+    <xacro:wheel_xacro wheel_name="right" xyz="0 -0.10 -0.06" />
+    <xacro:caster_xacro caster_name="front" xyz="0.08 0.0 -0.076" />
+    <xacro:caster_xacro caster_name="back" xyz="-0.08 0.0 -0.076" />
+    <!-- Gazebo 插件 -->
+    <xacro:include filename="$(find fishbot_description)/urdf/fishbot/plugins/gazebo_control_plugin.xacro" />
+    <!-- <xacro:gazebo_control_plugin /> -->
+    <xacro:include filename="$(find fishbot_description)/urdf/fishbot/fishbot.ros2_control.xacro" />
+    <xacro:fishbot_ros2_control />
+    <xacro:include filename="$(find fishbot_description)/urdf/fishbot/plugins/gazebo_sensor_plugin.xacro" />
+    <xacro:gazebo_sensor_plugin />
 </robot>

File: src/fishbot_description/urdf/fishbot/sensor/camera.urdf.xacro (robot description, xacro)
@@ -1,40 +1,39 @@
 <?xml version="1.0"?>
-<robot xmlns:xacro="http://www.ros.org/wiki/xacro" >
-    <xacro:include filename="$(find fishbot_description)/urdf/fishbot/common_inertia.xacro" />
+<robot xmlns:xacro="http://www.ros.org/wiki/xacro">
+   <xacro:include filename="$(find fishbot_description)/urdf/fishbot/common_inertia.xacro" />
     <xacro:macro name="camera_xacro" params="xyz">
-        <!-- 机器人相机部件 -->
+        <!-- ============相机模块================ -->
         <link name="camera_link">
             <visual>
-                <origin xyz="0 0 0" rpy="0 0 0" />
-                <geometry>
-                    <box size="0.02 0.10 0.02" />
-                </geometry>
-            <material name="black">
-                <color rgba="0 0 0 0.5" />
-            </material>
-            </visual>
-            <collision>
-                <origin xyz="0 0 0" rpy="0 0 0" />
+                <origin xyz="0 0 0.0" rpy="0 0 0" />
                 <geometry>
                     <box size="0.02 0.10 0.02" />
                 </geometry>
                 <material name="black">
-                <color rgba="0 0 0 0.5" />
-            </material>
+                    <color rgba="0.0 0.0 0.0 0.8"/>
+                </material>
+            </visual>
+            <collision>
+                <origin xyz="0 0 0.0" rpy="0 0 0" />
+                <geometry>
+                    <box size="0.02 0.10 0.02" />
+                </geometry>
+                <material name="black">
+                    <color rgba="0.0 0.0 0.0 0.8"/>
+                </material>
             </collision>
-        <xacro:box_inertia m="0.1"  w="0.10" h="0.02" d="0.02"/>
+            <xacro:box_inertia m="0.01" w="0.02" h="0.10" d="0.02" />
         </link>
-        <link name="camera_optical_link">
-        </link>
-    <joint name="camera_joint" type="fixed">
-        <origin xyz="${xyz}" rpy="0.0 0.0 0.0"/>
-        <parent link="base_link"/>
-        <child link="camera_link"/>
-    </joint>
-    <joint name="camera_optical_joint" type="fixed">
-        <parent link="camera_link"/>
-        <child link="camera_optical_link"/>
-        <origin xyz="0 0 0" rpy="${-pi/2} 0.0 ${-pi/2}"/>
-    </joint>
+        <link name="camera_optical_link"></link>
+        <joint name="camera_optical_joint" type="fixed">
+            <parent link="camera_link" />
+            <child link="camera_optical_link" />
+            <origin xyz="0 0 0" rpy="${-pi/2} 0 ${-pi/2}" />
+        </joint>
+        <joint name="camera_joint" type="fixed">
+            <parent link="base_link" />
+            <child link="camera_link" />
+            <origin xyz="${xyz}" />
+        </joint>
     </xacro:macro>
 </robot>

File: src/fishbot_description/urdf/fishbot/sensor/imu.urdf.xacro (robot description, xacro)
@@ -1,33 +1,32 @@
 <?xml version="1.0"?>
-<robot xmlns:xacro="http://www.ros.org/wiki/xacro" >
-    <xacro:include filename="$(find fishbot_description)/urdf/fishbot/common_inertia.xacro" />
+<robot xmlns:xacro="http://www.ros.org/wiki/xacro">
+   <xacro:include filename="$(find fishbot_description)/urdf/fishbot/common_inertia.xacro" />
     <xacro:macro name="imu_xacro" params="xyz">
-        <!-- 机器人IMU部件 -->
         <link name="imu_link">
             <visual>
-                <origin xyz="0 0 0" rpy="0 0 0" />
-                <geometry>
-                    <box size="0.02 0.02 0.02" />
-                </geometry>
-            <material name="black">
-                <color rgba="0 0 0 0.5" />
-            </material>
-            </visual>
-            <collision>
-                <origin xyz="0 0 0" rpy="0 0 0" />
+                <origin xyz="0 0 00" rpy="0 0 0" />
                 <geometry>
                     <box size="0.02 0.02 0.02" />
                 </geometry>
                 <material name="black">
-                    <color rgba="0 0 0 0.5" />
+                    <color rgba="0 0 0 0.8" />
+                </material>
+            </visual>
+            <collision>
+                <origin xyz="0 0 00" rpy="0 0 0" />
+                <geometry>
+                    <box size="0.02 0.02 0.02" />
+                </geometry>
+                <material name="black">
+                    <color rgba="0 0 0 0.8" />
                 </material>
             </collision>
-            <xacro:box_inertia m="0.05" w="0.02" h="0.02" d="0.02"/>
+            <xacro:box_inertia m="0.01" w="0.02" d="0.02" h="0.02"/>
         </link>
-    <joint name="imu_joint" type="fixed">
-        <origin xyz="${xyz}" rpy="0.0 0.0 0.0"/>
-        <parent link="base_link"/>
-        <child link="imu_link"/>
-    </joint>
+        <joint name="imu_joint" type="fixed">
+            <parent link="base_link" />
+            <child link="imu_link" />
+            <origin xyz="${xyz}" />
+        </joint>
     </xacro:macro>
 </robot>

File: src/fishbot_description/urdf/fishbot/sensor/laser.urdf.xacro (robot description, xacro)
@@ -1,36 +1,21 @@
 <?xml version="1.0"?>
-<robot xmlns:xacro="http://www.ros.org/wiki/xacro" >
-    <xacro:include filename="$(find fishbot_description)/urdf/fishbot/common_inertia.xacro" />
+<robot xmlns:xacro="http://www.ros.org/wiki/xacro">
+   <xacro:include filename="$(find fishbot_description)/urdf/fishbot/common_inertia.xacro" />
     <xacro:macro name="laser_xacro" params="xyz">
-        <!-- 机器人激光雷达部件 -->
+        <gazebo reference="laser_cylinder_link">
+            <material>Gazebo/Black</material>
+        </gazebo>
+        <gazebo reference="laser_link">
+            <material>Gazebo/Black</material>
+        </gazebo>
+        <!-- ============雷达支撑杆================ -->
         <link name="laser_cylinder_link">
             <visual>
                 <origin xyz="0 0 0" rpy="0 0 0" />
                 <geometry>
-                    <cylinder radius="0.01" length="0.1" />
-                </geometry>
-            <material name="black">
-                <color rgba="0 0 0 1.0" />
-            </material>
-            </visual>
-            <collision>
-                <origin xyz="0 0 0" rpy="0 0 0" />
-                <geometry>
-                    <cylinder radius="0.01" length="0.1" />
+                    <cylinder length="0.10" radius="0.01" />
                 </geometry>
                 <material name="black">
-                    <color rgba="0 0 0 1.0" />
-                </material>
-            </collision>
-            <xacro:cylinder_inertia m="0.05" r="0.01" h="0.1" />
-        </link>
-        <link name="laser_link">
-            <visual>
-                <origin xyz="0 0 0" rpy="0 0 0" />
-                <geometry>
-                    <cylinder radius="0.02" length="0.02" />
-                </geometry>
-                <material name="red">
-                    <color rgba="1 0 0 1.0" />
+                    <color rgba="0.0 0.0 0.0 0.8" />
                 </material>
             </visual>
@@ -38,30 +23,44 @@
                 <origin xyz="0 0 0" rpy="0 0 0" />
                 <geometry>
-                    <cylinder radius="0.02" length="0.02" />
+                    <cylinder length="0.10" radius="0.01" />
                 </geometry>
-                <material name="red">
-                    <color rgba="1 0 0 1.0" />
+                <material name="black">
+                    <color rgba="0.0 0.0 0.0 0.8" />
                 </material>
             </collision>
-            <xacro:cylinder_inertia m="0.05" r="0.02" h="0.02" />
+            <xacro:cylinder_inertia m="0.01" r="0.01" h="0.10" />
         </link>
-    <!-- 激光雷达to圆柱关节 -->
-    <joint name="laser_joint" type="fixed">
-        <parent link="laser_cylinder_link"/>
-        <child link="laser_link"/>
-        <origin xyz="0.0 0.0 0.05" rpy="0.0 0.0 0.0"/>
-    </joint>
-    <!-- 激光雷达to基座关节 -->
-    <joint name="laser_cylinder_joint" type="fixed">
-        <parent link="base_link"/>
-        <child link="laser_cylinder_link"/>
-        <origin xyz="${xyz}" rpy="0.0 0.0 0.0"/>
-    </joint>
-    <gazebo reference="laser_cylinder_link">
-        <material>Gazebo/Black</material>
-    </gazebo>
-    <gazebo reference="laser_link">
-        <material>Gazebo/Red</material>
-    </gazebo>
+        <joint name="laser_cylinder_joint" type="fixed">
+            <parent link="base_link" />
+            <child link="laser_cylinder_link" />
+            <origin xyz="${xyz}" />
+        </joint>
+        <!-- ============雷达================ -->
+        <link name="laser_link">
+            <visual>
+                <origin xyz="0 0 0" rpy="0 0 0" />
+                <geometry>
+                    <cylinder length="0.02" radius="0.02" />
+                </geometry>
+                <material name="black">
+                    <color rgba="0.0 0.0 0.0 0.8" />
+                </material>
+            </visual>
+            <collision>
+                <origin xyz="0 0 0" rpy="0 0 0" />
+                <geometry>
+                    <cylinder length="0.02" radius="0.02" />
+                </geometry>
+                <material name="black">
+                    <color rgba="0.0 0.0 0.0 0.8" />
+                </material>
+            </collision>
+            <xacro:cylinder_inertia m="0.03" r="0.02" h="0.02" />
+        </link>
+        <joint name="laser_joint" type="fixed">
+            <parent link="laser_cylinder_link" />
+            <child link="laser_link" />
+            <origin xyz="0 0 0.05" />
+        </joint>
     </xacro:macro>
 </robot>
